Commit message: Flushed out Walker a little

File: Robots/Prototype/Prototype.urdf (robot description, URDF)
Before this commit: robot Prototype, 22 links, 21 joints
Joints:
- joint right_aiming_hip: origin xyz=0.312 -0.67 -0.06 rpy=6.28318530718 0.0 -1.57079632679 -> xyz=0.3125 -0.67 -0.06 rpy=6.28318530718 0.0 -1.57079632679
- joint right_aiming_hip_servo: origin xyz=0.312 -0.67 -0.06 rpy=3.14159265359 0.0 -1.57079632679 -> xyz=0.3125 -0.67 -0.06 rpy=3.14159265359 0.0 -1.57079632679

File: Robots/Prototype/Prototype.urdf.xacro (robot description, xacro)
@@ -144,4 +144,4 @@
 	<xacro:leg name="back" thighL="0.94" calfL="0.93" xyz="-0.75 0 ${-servoD/2}" ydeg="180"/>
 	<xacro:leg name="left" thighL="0.91" calfL="0.94" xyz="0.3125 ${popsicleL/2 + hornD + servoL2} ${-servoD/2}" ydeg="90"/>
-	<xacro:leg name="right" thighL="0.92" calfL="0.93" xyz="0.312 ${-popsicleL/2 - hornD - servoL2} ${-servoD/2}" ydeg="-90" reflect="-1"/>
+	<xacro:leg name="right" thighL="0.92" calfL="0.93" xyz="0.3125 ${-popsicleL/2 - hornD - servoL2} ${-servoD/2}" ydeg="-90" reflect="-1"/>
 </robot>
