Commit message: Basic walking.  Implementation may be a little overcomplex.

File: Robots/B_Hunker/Hunker.urdf (robot description, URDF)
Before this commit: robot Hunker, 17 links, 16 joints
Joints:
- joint backLeftAnkle: origin xyz=-0.33 0.12 0 -> xyz=-0.24 0.12 0
- joint backRightAnkle: origin xyz=-0.33 -0.12 0 -> xyz=-0.24 -0.12 0
- joint frontLeftAnkle: origin xyz=-0.33 0.12 0 -> xyz=-0.24 0.12 0
- joint frontRightAnkle: origin xyz=-0.33 -0.12 0 -> xyz=-0.24 -0.12 0

File: Robots/B_Hunker/Hunker.urdf.xacro (robot description, xacro)
@@ -104,11 +104,11 @@
 		</joint>
 		<link name="${name}Foot">
-			<xacro:wheelY x="1.5" y="2.25" z="0"><xacro:mud/></xacro:wheelY>
-			<xacro:wheelY x="1.5" y="-2.25" z="0"><xacro:mud/></xacro:wheelY>
+			<xacro:wheelY x="0" y="2.25" z="0"><xacro:mud/></xacro:wheelY>
+			<xacro:wheelY x="0" y="-2.25" z="0"><xacro:mud/></xacro:wheelY>
 		</link>
 		<joint name="${name}Ankle" type="fixed">
 			<parent link="${name}Calf"/>
 			<child link="${name}Foot"/>
-			<origin xyz="${-5.5 * pitch} ${-2 * reflect * pitch} 0"/>
+			<origin xyz="${-4 * pitch} ${-2 * reflect * pitch} 0"/>
 		</joint>
 	</xacro:macro>
